File: hardware/ldo-power-board/ldo-power-board.kicad_pcb (KiCad board)
At the start: 2 copper layers, 25.4 x 25.4 mm, 13 parts, among them J1 Conn_01x02, J2 Conn_01x04, U1 ADP322ACPZ-135-R7

Commit message: Done with da layout
Parts:
- added H3: MountingHole, MountingHole:MountingHole_2.1mm, F.Cu at (152.4, 111.8)
- added H4: MountingHole, MountingHole:MountingHole_2.1mm, F.Cu at (152.4, 91.4)
- U1: value ADP322ACPZ-135-R7 -> CP_16_22_ADI
- moved FID1 41.8 mm to (134.6, 95.2)
- moved U1 30.5 mm to (142.2, 101.6)
- moved H1 26.0 mm to (132.1, 91.4)
- moved C1 25.8 mm to (144.3, 105.9), turned to 270 degrees
- moved C2 25.2 mm to (142.2, 105.9), turned to 270 degrees
- moved FID2 24.6 mm to (149.9, 108.0)
- moved C3 22.6 mm to (140.7, 105.9), turned to 270 degrees
- moved C6 20.9 mm to (146.1, 101.6), turned to 90 degrees
- moved C5 17.3 mm to (138.2, 103.4), turned to 270 degrees
- moved C4 17.1 mm to (138.2, 99.8), turned to 90 degrees
- moved H2 11.3 mm to (132.1, 111.8)
- moved J1 6.37 mm to (130.8, 100.3)
- moved J2 6.00 mm to (153.7, 97.8)
Routing:
- net /VIN: track 0.12 -> 35.7 mm
- net /VOUT1: track 0.00 -> 20.3 mm, vias 0 -> 1
- net /VOUT2: track 0.00 -> 15.5 mm, vias 0 -> 1
- net /VOUT3: track 0.00 -> 12.8 mm
- net GND: track 0.00 -> 1.04 mm, vias 0 -> 31
- added copper zone on B.Cu, net GND
- added copper zone on F.Cu, net GND
Other:
- net class Default: clearance 0.22 -> 0.2032
- net class Power: clearance 0.22 -> 0.2032; trace_width 0.3 -> 0.381
- rule trace_clearance: 0.22 -> 0.2032
- board text added: "ADP322 Fixed Voltage"
- board text added: "GND"
- board text added: "LDO Power Breakout Board"
- board text added: "VIN"
- board text added: "VIN Range: 2.5-5.5V 200 mA max each VOUT"
- board text added: "VOUT1"
- board text added: "VOUT2"
- board text added: "VOUT3"
- board text added: "v01"
